Commit message: S

File: tm_description/xacro/tm12.ros2_control.xacro (robot description, xacro)
@@ -1,10 +1,10 @@
 <?xml version="1.0"?>
 <robot xmlns:xacro="http://www.ros.org/wiki/xacro">
-    <xacro:macro name="tm12_ros2_control" params="name">
+    <xacro:macro name="tm12_ros2_control" params="name prefix">
         <ros2_control name="${name}" type="system">
             <hardware>
                 <plugin>tm_robot_driver/TMPositionHardwareInterface</plugin>
             </hardware>
-            <joint name="joint_1">
+            <joint name="${prefix}joint_1">
                 <command_interface name="position">
                     <param name="min">${radians(-270)}</param>
@@ -16,5 +16,5 @@
                 <state_interface name="effort"/>
             </joint>
-            <joint name="joint_2">
+            <joint name="${prefix}joint_2">
                 <command_interface name="position">
                     <param name="min">${radians(-180)}</param>
@@ -26,5 +26,5 @@
                 <state_interface name="effort"/>
             </joint>
-            <joint name="joint_3">
+            <joint name="${prefix}joint_3">
                 <command_interface name="position">
                     <param name="min">${radians(-166)}</param>
@@ -36,5 +36,5 @@
                 <state_interface name="effort"/>
             </joint>
-            <joint name="joint_4">
+            <joint name="${prefix}joint_4">
                 <command_interface name="position">
                     <param name="min">${radians(-180)}</param>
@@ -46,5 +46,5 @@
                 <state_interface name="effort"/>
             </joint>
-            <joint name="joint_5">
+            <joint name="${prefix}joint_5">
                 <command_interface name="position">
                     <param name="min">${radians(-180)}</param>
@@ -56,5 +56,5 @@
                 <state_interface name="effort"/>
             </joint>
-            <joint name="joint_6">
+            <joint name="${prefix}joint_6">
                 <command_interface name="position">
                     <param name="min">${radians(-270)}</param>

File: tm_description/xacro/tm12.urdf.xacro (robot description, xacro)
@@ -16,4 +16,7 @@
   <xacro:tmr_transmission prefix="$(arg prefix)" hw_iface="$(arg trans_hw_iface)" />
   <xacro:tmr_materials/>
+  <!-- ros2 control include -->
+  <xacro:include filename="$(find tm_description)/xacro/tm12.ros2_control.xacro" />
+  <xacro:tm12_ros2_control name="tm12" />
   <!-- Arm -->
   <xacro:property name="color" value="$(arg color)"/>

Commit message: Add mock hardware interface

File: tm_description/xacro/tm12.ros2_control.xacro (robot description, xacro)
@@ -1,8 +1,13 @@
 <?xml version="1.0"?>
 <robot xmlns:xacro="http://www.ros.org/wiki/xacro">
-    <xacro:macro name="tm12_ros2_control" params="name prefix">
+    <xacro:macro name="tm12_ros2_control" params="name prefix use_fake_hardware:=false">
         <ros2_control name="${name}" type="system">
             <hardware>
+              <xacro:if value="${use_fake_hardware}">
+                <plugin>mock_components/GenericSystem</plugin>
+              </xacro:if>
+              <xacro:unless value="${use_fake_hardware}">
                 <plugin>tm_robot_driver/TMPositionHardwareInterface</plugin>
+              </xacro:unless>
             </hardware>
             <joint name="${prefix}joint_1">
